File: BME280_PCB/BME280_PCB.kicad_pcb (KiCad board)
At the start: 2 copper layers, 6 parts, among them J1 110990030, U5 BME280

Commit message: Finished all PCBs, initial CAD complete
Parts:
- removed J1: 110990030, ExternalFootprints:SEEED_110990030
- removed U5: BME280, Package_LGA:Bosch_LGA-8_2.5x2.5mm_P0.65mm_ClockwisePinNumbering
- added J2: Screw_Terminal_01x04, TerminalBlock_Phoenix:TerminalBlock_Phoenix_MKDS-1,5-4_1x04_P5.00mm_Horizontal, F.Cu at (22.1, 20.7)
- added U1: BME280, Package_LGA:Bosch_LGA-8_2.5x2.5mm_P0.65mm_ClockwisePinNumbering, F.Cu at (12.3, 12.1)
- moved C2 110.6 mm to (10.1, 13.1), turned to -90 degrees
- moved C1 109.8 mm to (10.1, 11.2), turned to -90 degrees
- moved R1 106.8 mm to (14.4, 13.6), turned to 90 degrees
- moved R2 104.9 mm to (14.4, 11.6), turned to -90 degrees
Routing:
- net +3V3: track 0.00 -> 24.3 mm
- net /BME280_SDA: track 0.00 -> 11.7 mm, vias 0 -> 1
- net /BME280_SCL: track 0.00 -> 9.91 mm, vias 0 -> 1
- net GND: track 0.00 -> 4.41 mm, vias 0 -> 4
- added copper zone on B.Cu, net GND
Other:
- board outline added: 18.9 x 21.1 mm
- board text added: "GND"
- board text added: "SCL"
- board text added: "SDA"
- board text added: "VIN"
