File: BME280_PCB/BME280_PCB.kicad_sch (KiCad schematic)
At the start: 6 parts, among them J1 110990030, U5 BME280

Commit message: Finished all PCBs, initial CAD complete
Parts:
- removed J1: 110990030, ExternalFootprints:SEEED_110990030, symbol Grove_4P_Connector:110990030
- added J2: Screw_Terminal_01x04, TerminalBlock_Phoenix:TerminalBlock_Phoenix_MKDS-1,5-4_1x04_P5.00mm_Horizontal, symbol Connector:Screw_Terminal_01x04
- renumbered U5 to U1
Connections:
- net +3V3: now also J2.1 (Pin_1); no longer U1.5 (SDO)
- net BME280_SCL: now also J2.3 (Pin_3)
- net BME280_SDA: now also J2.4 (Pin_4)
- net GND: now also U1.5 (SDO), J2.2 (Pin_2)
Other:
- note removed: "GND"
- note removed: "SCL"
- note removed: "SDA"
- note removed: "VCC"
