File: MAIN_PCB/Plant Monitor.kicad_pcb (KiCad board)
At the start: 2 copper layers, 0.7 x 0.6 mm, 59 parts, among them J1 USB4235-03-C_REVA, J2 Motor 1, J3 Motor 2, J4 Grove Connector for Soil Mois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, J5 JST PH-2Pin, J6 Grove Connector for OLED Disp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, J7 Conn_01x15, J8 Conn_01x15, Q1 AO3401A, SW1 SW_Push, SW2 SW_Push, U1 RP2040, U2 AP2112K-3.3, U3 DRV8833CPWPR, U4 W25Q128JVS, U5 BME280, U6 MCP73831-2-OT, X1 ABM8-272-T3

Commit message: Updated PCB design+schematic
Parts:
- removed C22, C23: 0.1uF, Capacitor_SMD:C_0402_1005Metric
- removed J7: Conn_01x15, Connector_PinHeader_2.54mm:PinHeader_1x15_P2.54mm_Vertical
- removed R16: 4.7k, Resistor_SMD:R_0402_1005Metric
- removed U5: BME280, Package_LGA:Bosch_LGA-8_2.5x2.5mm_P0.65mm_ClockwisePinNumbering
- added D3: Green, LED_SMD:LED_0603_1608Metric, F.Cu at (220.9, 76.6)
- added D4: Green, LED_SMD:LED_0603_1608Metric, F.Cu at (222.7, 76.6)
- added J10: BME280 Terminals, TerminalBlock_Phoenix:TerminalBlock_Phoenix_MKDS-1,5-4_1x04_P5.00mm_Horizontal, F.Cu at (240.1, 66.3)
- added R14: 330, Resistor_SMD:R_0402_1005Metric, F.Cu at (220.9, 73.9)
- C11: value 1uF -> 0.1uF
- C2, C3, C6, Q1: moved to B.Cu
- C4, C9: value 0.1uF -> 1uF
- C8: value 1uF -> 0.1uF; moved to B.Cu
- D2: footprint LED_SMD:LED_0402_1005Metric -> LED_SMD:LED_0603_1608Metric
- J1: value USB4235-03-C_REVA -> TYPE-C-31-M-12; footprint ExternalFootprints:GCT_USB4235-03-C_REVA -> ExternalFootprints:HRO_TYPE-C-31-M-12
- J3: footprint TerminalBlock_Phoenix:TerminalBlock_Phoenix_MKDS-1,5-2-5.08_1x02_P5.08mm_Horizontal -> Connector_PinHeader_2.54mm:PinHeader_1x02_P2.54mm_Vertical
- J8: footprint Connector_PinHeader_2.54mm:PinHeader_1x15_P2.54mm_Vertical -> Connector_PinHeader_2.54mm:PinHeader_1x11_P2.54mm_Vertical
- R11: value 10k -> 470
- R15: value 4.7k -> 500
- R3, R4: value 1 -> 0.2
- U1: footprint Package_DFN_QFN:QFN-56-1EP_7x7mm_P0.4mm_EP3.2x3.2mm -> Package_DFN_QFN:QFN-56-1EP_7x7mm_P0.4mm_EP3.2x3.2mm_ThermalVias
- U3: value DRV8833CPWPR -> DRV8833PWP; footprint ExternalFootprints:SOP65P640X120-17N -> Package_SO:HTSSOP-16-1EP_4.4x5mm_P0.65mm_EP3.4x5mm_Mask2.46x2.31mm_ThermalVias
- U4: value W25Q128JVS -> W25Q16JVSS; footprint Package_SO:SOIC-8_5.3x5.3mm_P1.27mm -> Package_SON:Winbond_USON-8-1EP_3x2mm_P0.5mm_EP0.2x1.6mm
- moved J8 107.7 mm to (244.0, 99.6)
- moved SW1 87.9 mm to (237.4, 99.5), turned to -45 degrees
- moved J2 84.7 mm to (214.8, 121.0), turned to 180 degrees
- moved C4 84.1 mm to (229.0, 85.1), turned to 90 degrees
- moved C6 81.7 mm to (230.1, 87.7)
- moved C7 81.4 mm to (229.9, 91.2)
- moved C5 81.3 mm to (229.7, 86.7)
- moved C2 81.2 mm to (226.5, 84.7), turned to 90 degrees
- moved C21 80.9 mm to (235.1, 95.4), turned to 135 degrees
- moved C3 80.4 mm to (225.5, 84.7), turned to 90 degrees
- moved J4 80.4 mm to (240.4, 87.4)
- moved C9 80.1 mm to (227.8, 85.1), turned to 90 degrees
- moved C8 76.5 mm to (224.9, 96.1), turned to -90 degrees
- moved C11 75.7 mm to (226.8, 96.0), turned to -90 degrees
- moved C16 75.5 mm to (226.9, 97.8), turned to -90 degrees
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Connections:
- C0 pad 2: +1V1 -> GND
- C1 pad 2: +1V1 -> GND
- C10 pad 2: +1V1 -> GND
- C11 pad 2: +1V1 -> GND
- C12 pad 1: Net-(D1-K) -> /+MOTORVOLTAGE
- C12 pad 2: +1V1 -> GND
- C13 pad 2: +1V1 -> GND
- C14 pad 2: +1V1 -> GND
- C15 pad 1: +5V -> /+MOTORVOLTAGE
- C15 pad 2: +1V1 -> GND
- C16 pad 2: +1V1 -> GND
- C17 pad 2: +1V1 -> GND
- C18 pad 2: +1V1 -> GND
- C19 pad 1: +1V1 -> +BATT
- C19 pad 2: +1V1 -> GND
- C2 pad 2: +1V1 -> GND
- C20 pad 2: +1V1 -> GND
- C21 pad 2: +1V1 -> GND
- C3 pad 2: +1V1 -> GND
- C4 pad 2: +1V1 -> GND
- C5 pad 2: +1V1 -> GND
- C6 pad 2: +1V1 -> GND
- C7 pad 2: +1V1 -> GND
- C8 pad 2: +1V1 -> GND
- C9 pad 2: +1V1 -> GND
- D1 pad 1: Net-(D1-K) -> /+MOTORVOLTAGE
- J4 pad 1: +1V1 -> /SOIL_SIG
- J4 pad 2: +3V3 -> unconnected-(J4-Pad2)
- J4 pad 3: /SOIL_DISABLE -> +3V3
- J4 pad 4: /SOIL_OUT -> GND
- J5 pad 1: +1V1 -> +BATT
- J5 pad 2: +1V1 -> GND
- J6 pad 1: +1V1 -> /OLED_SCL
- J6 pad 2: +3V3 -> /OLED_SDA
- J6 pad 3: /OLED_SDA -> +3V3
- J6 pad 4: /OLED_SCL -> GND
- J8 pad 1: +3V3 -> /GPIO28/ADC0
- J8 pad 10: /GPIO26/ADC0 -> +3V3
- J8 pad 11: /GPIO27/ADC1 -> GND
- J8 pad 2: /SWCLK -> /GPIO27/ADC1
- J8 pad 3: +1V1 -> /GPIO27/ADC2
- J8 pad 4: /GPIO16 -> /GPIO15
- J8 pad 5: /GPIO17 -> /GPIO16
- J8 pad 6: /GPIO18 -> /GPIO17
- J8 pad 7: /GPIO19 -> /GPIO18
- J8 pad 8: /GPIO20 -> /GPIO19
- J8 pad 9: /GPIO21 -> +3V3
- Q1 pad 2: Net-(D1-K) -> /+MOTORVOLTAGE
- Q1 pad 3: +1V1 -> +BATT
- R10 pad 2: +1V1 -> GND
- R11 pad 1: Net-(U6-STAT) -> Net-(D2-K)
- R11 pad 2: Net-(D2-K) -> Net-(U6-STAT)
- R12 pad 2: +1V1 -> GND
- R15 pad 1: +3V3 -> Net-(D4-K)
- R15 pad 2: /BME280_SDA -> GND
- R3 pad 1: +1V1 -> GND
- R4 pad 1: +1V1 -> GND
- R6 pad 1: Net-(J1-CC2) -> Net-(J1-CC1)
- R6 pad 2: +1V1 -> GND
- R7 pad 1: Net-(J1-CC1) -> Net-(J1-CC2)
- R7 pad 2: +1V1 -> GND
- SW1 pad 2: +1V1 -> GND
- SW2 pad 2: +1V1 -> GND
- U1 pad 19: +1V1 -> GND
- U1 pad 24: /SWCLK -> unconnected-(U1-SWCLK-Pad24)
- U1 pad 25: /SWDIO -> unconnected-(U1-SWDIO-Pad25)
- U1 pad 31: /GPIO20 -> /BME280_SCL
- U1 pad 32: /GPIO21 -> /BME280_SDA
- U1 pad 34: /SOIL_DISABLE -> /GPIO22
- U1 pad 35: /SOIL_OUT -> /GPIO23
- U1 pad 38: /GPIO26/ADC0 -> /GPIO28/ADC0
- U1 pad 40: /GPIO28/ADC2 -> /GPIO27/ADC2
- U1 pad 41: /GPIO29/ADC3 -> /SOIL_SIG
- U1 pad 57: +1V1 -> GND
- U2 pad 1: Net-(D1-K) -> /+MOTORVOLTAGE
- U2 pad 2: +1V1 -> GND
- U2 pad 3: Net-(D1-K) -> /+MOTORVOLTAGE
- U3 pad 11: (no net) -> GND
- U3 pad 12: +5V -> /+MOTORVOLTAGE
- U3 pad 13: +1V1 -> GND
- U3 pad 17: unconnected-(U3-EXP-Pad17) -> GND
- U4 pad 4: +1V1 -> GND
- U6 pad 2: +1V1 -> GND
- U6 pad 3: +1V1 -> +BATT
- X1 pad 2: +1V1 -> GND
- X1 pad 4: +1V1 -> GND
Routing:
- net /nSLEEP: track 0.00 -> 46.0 mm, vias 0 -> 2
- net /nFAULT: track 0.00 -> 39.0 mm, vias 0 -> 2
- net +5V: track 0.00 -> 36.3 mm, vias 0 -> 3
- net /GPIO19: track 0.00 -> 31.8 mm, vias 0 -> 1
- net /GPIO18: track 0.00 -> 28.5 mm, vias 0 -> 1
- net /GPIO27/ADC2: track 0.00 -> 27.9 mm, vias 0 -> 2
- net /GPIO15: track 0.00 -> 27.3 mm, vias 0 -> 2
- net /GPIO17: track 0.00 -> 26.3 mm, vias 0 -> 1
- net /GPIO27/ADC1: track 0.00 -> 25.2 mm, vias 0 -> 2
- net /GPIO16: track 0.00 -> 24.7 mm, vias 0 -> 1
- net /+MOTORVOLTAGE: track 0.00 -> 23.4 mm, vias 0 -> 3
- net /BME280_SDA: track 0.00 -> 23.1 mm, vias 0 -> 2
- net +3V3: track 0.00 -> 22.6 mm, vias 0 -> 7
- net /GPIO28/ADC0: track 0.00 -> 22.3 mm, vias 0 -> 2
- net /BME280_SCL: track 0.00 -> 21.6 mm, vias 0 -> 2
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- added copper zone on In2.Cu, net /+MOTORVOLTAGE
- added copper zone on In1.Cu, net GND
Other:
- board size 0.7 x 0.6 mm -> 42.8 x 66.3 mm
- copper layers 2 -> 4

Commit message: Finished main PCB
Parts:
- removed C21: 0.1uF, Capacitor_SMD:C_0402_1005Metric
- removed the J8 at (244.0, 99.6)
- removed the SW1 at (237.4, 99.5)
- added J6: Conn_01x14, Connector_PinHeader_2.54mm:PinHeader_1x14_P2.54mm_Vertical, F.Cu at (244.0, 91.7)
- added J7: Conn_01x14, Connector_PinHeader_2.54mm:PinHeader_1x14_P2.54mm_Vertical, F.Cu at (204.8, 77.6)
- C11, R13, R3, R4: moved to B.Cu
- moved J5 28.1 mm to (236.7, 95.0), turned to -90 degrees
- moved J2 13.1 mm to (227.9, 121.0)
- moved R15 7.83 mm to (230.0, 71.0)
- moved D3 7.83 mm to (228.2, 73.7)
- moved D4 7.83 mm to (230.0, 73.7)
- moved R14 7.83 mm to (228.2, 71.0)
- moved R3 6.82 mm to (213.2, 120.3)
- moved R4 6.25 mm to (215.7, 119.5), turned to 180 degrees
- moved U3 6.18 mm to (214.2, 114.4)
- moved C14 6.18 mm to (213.2, 108.8)
- moved C15 6.18 mm to (214.8, 107.3)
- moved SW1 5.85 mm to (214.1, 90.3), turned to -90 degrees
- moved J3 5.57 mm to (204.8, 116.4)
- moved R13 4.59 mm to (229.3, 93.9), turned to 180 degrees
- moved C11 4.15 mm to (224.2, 92.7), turned to 180 degrees
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- renumbered J6 to J5, J5 to J8, J10 to J9, SW2 to SW1, U6 to U5
Connections:
- net /RUN renamed Net-(U1-RUN)
- U1 pad 24: unconnected-(U1-SWCLK-Pad24) -> /SWCLK
- U1 pad 25: unconnected-(U1-SWDIO-Pad25) -> /SWDIO
- U1 pad 34: /GPIO22 -> /nFAULT
- U1 pad 35: /GPIO23 -> /nSLEEP
- U1 pad 36: /nSLEEP -> /OLED_SDA
- U1 pad 37: /nFAULT -> /OLED_SCL
- U1 pad 38: /GPIO28/ADC0 -> /GPIO26/ADC0
- U1 pad 40: /GPIO27/ADC2 -> /GPIO28/ADC2
- U1 pad 6: /OLED_SDA -> /GPIO4
- U1 pad 7: /OLED_SCL -> /GPIO5
- U4 pad 9: (no net) -> GND
Routing:
- net /GPIO27/ADC2: track 27.9 -> 0.00 mm, vias 2 -> 0
- net /SWCLK: track 0.00 -> 27.0 mm
- net /SWDIO: track 0.00 -> 24.9 mm
- net GND: track 11.2 -> 34.9 mm, vias 38 -> 61
- net /GPIO14: track 0.00 -> 22.4 mm, vias 0 -> 1
- net /GPIO28/ADC0: track 22.3 -> 0.00 mm, vias 2 -> 0
- net /GPIO0: track 0.00 -> 21.8 mm
- net /GPIO8: track 0.00 -> 21.4 mm, vias 0 -> 1
- net /GPIO26/ADC0: track 0.00 -> 20.3 mm, vias 0 -> 1
- net /GPIO1: track 0.00 -> 20.2 mm
- net /GPIO9: track 0.00 -> 20.0 mm
- net /GPIO2: track 0.00 -> 19.3 mm
- net /GPIO7: track 0.00 -> 18.4 mm, vias 0 -> 1
- net /GPIO3: track 0.00 -> 18.4 mm
- net /GPIO28/ADC2: track 0.00 -> 18.3 mm, vias 0 -> 1
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- added copper zone on In2.Cu, net +3V3
- added copper zone on In3.Cu, net /+MOTORVOLTAGE
- added copper zone on F.Cu, net GND
- added copper zone on In4.Cu, net GND
- removed copper zone on In2.Cu, net /+MOTORVOLTAGE
Other:
- copper layers 4 -> 6
- board text added: "+3V3"
- board text added: "+MOTOR"
- board text added: "+V"
- board text added: "0"
- board text added: "1"
- board text added: "14"
- board text added: "15"
- board text added: "16"
- board text added: "17"
- board text added: "18"
- board text added: "19"
- board text added: "2"
- board text added: "26"
- board text added: "27"
- board text added: "28"
- board text added: "3"
- board text added: "3V3"
- board text added: "4"
- board text added: "5"
- board text added: "6"
- board text added: "7"
- board text added: "8"
- board text added: "9"
- board text added: "A1"
- board text added: "A2"
- board text added: "All vias that are in pads and have a total diameter of 24 mils and hole diameter 10 mils should be filled with epoxy and capped over (IPC-4761 Type VII via) All vias within copper pours should also be filled with epoxy for thermal conductivity"
- board text added: "B1"
- board text added: "B2"
- board text added: "CYUE"
- board text added: "GND"
- board text added: "P-MON V1.0"
- board text added: "SCL"
- board text added: "SDA"
- board text added: "SIG"
- board text added: "SWCLK"
- board text added: "SWDIO"
- board text added: "~"

Commit message: Finished main PCB
Parts:
- added ?: , clipboard:0abc01f6-72ea-4eb5-a1fb-07ac69a68b80, F.Cu at (217.2, 79.1)
- added ?: , clipboard:0abc01f6-72ea-4eb5-a1fb-07ac69a68b80, F.Cu at (223.2, 99.7)
- added ?: , clipboard:0abc01f6-72ea-4eb5-a1fb-07ac69a68b80, F.Cu at (211.6, 71.0)
- added ?: , clipboard:0abc01f6-72ea-4eb5-a1fb-07ac69a68b80, F.Cu at (237.3, 83.9)
- added ?: , clipboard:0abc01f6-72ea-4eb5-a1fb-07ac69a68b80, F.Cu at (233.8, 92.1)
- added ?: , clipboard:0abc01f6-72ea-4eb5-a1fb-07ac69a68b80, F.Cu at (205.6, 65.7)
- added SW2: SW_Push, Button_Switch_SMD:SW_Tactile_SPST_NO_Straight_CK_PTS636Sx25SMTRLFS, F.Cu at (228.8, 106.6)
- moved SW1 1.85 mm to (212.3, 90.3)
- moved R9 1.85 mm to (214.1, 86.1)
- moved C12 0.60 mm to (218.7, 78.4)
- moved C0 0.41 mm to (218.6, 87.6)
Connections:
- net Net-(U1-RUN) renamed /RUN
Routing:
- net /RUN: track 3.10 -> 12.2 mm, vias 1 -> 2
- net /QSPI_SS: track 11.0 -> 12.9 mm
- net GND: track 34.9 -> 36.3 mm, vias 61 -> 62
- net /+MOTORVOLTAGE: track 24.7 -> 25.4 mm
- net /GPIO5: track 16.7 -> 17.2 mm, vias 0 -> 1
- net /GPIO0: track 21.8 -> 21.4 mm, vias 0 -> 1
- net /GPIO4: track 17.5 -> 17.6 mm, vias 0 -> 1
- net /GPIO3: vias 0 -> 1
- net /GPIO6: vias 0 -> 1
- net /GPIO2: vias 0 -> 1
- net /GPIO1: vias 0 -> 1
Other:
- board text added: "BOOT"
- board text added: "RESET"

Commit message: Finished all PCBs, initial CAD complete
Parts:
- removed ? (x6): , clipboard:0abc01f6-72ea-4eb5-a1fb-07ac69a68b80
- moved J2 216.7 mm to (19.7, 61.2), turned to 0 degrees
- moved C0 211.8 mm to (15.6, 27.2)
- moved C10 211.8 mm to (21.3, 23.2)
- moved C11 211.8 mm to (21.3, 32.3)
- moved C13 211.8 mm to (13.3, 22.4)
- moved C14 211.8 mm to (10.3, 48.4)
- moved C15 211.8 mm to (11.9, 46.9)
- moved C16 211.8 mm to (23.9, 37.4)
- moved C17 211.8 mm to (18.4, 37.4)
- moved C19 211.8 mm to (9.27, 7.80)
- moved C3 211.8 mm to (22.1, 24.1)
- moved C4 211.8 mm to (26.1, 24.7)
- moved C7 211.8 mm to (27.6, 30.7)
- moved C9 211.8 mm to (24.9, 24.7)
- moved D1 211.8 mm to (14.1, 9.38)
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Connections:
- J9 pad 1: +3V3 -> /BME280_SDA
- J9 pad 2: GND -> /BME280_SCL
- J9 pad 3: /BME280_SDA -> +3V3
- J9 pad 4: /BME280_SCL -> GND
- U1 pad 31: /BME280_SCL -> /BME280_SDA
- U1 pad 32: /BME280_SDA -> /BME280_SCL
- U3 pad 2: Net-(J2-Pin_1) -> Net-(J2-Pin_2)
- U3 pad 4: Net-(J2-Pin_2) -> Net-(J2-Pin_1)
Routing:
- net Net-(J2-Pin_1): track 21.7 -> 11.5 mm
- net Net-(J2-Pin_2): track 12.0 -> 21.0 mm
- net /BME280_SCL: track 23.4 -> 25.5 mm
- net /BME280_SDA: track 25.3 -> 23.7 mm
- net GND: track 36.3 -> 35.0 mm
- net +5V: track 38.0 -> 37.1 mm
