File: MAIN_PCB/Plant Monitor.kicad_sch (KiCad schematic)
At the start: 59 parts, among them J1 USB4235-03-C_REVA, J2 Motor 1, J3 Motor 2, J4 Grove Connector for Soil Mois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, J5 JST PH-2Pin, J6 Grove Connector for OLED Disp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, J7 Conn_01x15, J8 Conn_01x15, Q1 AO3401A, SW1 SW_Push, SW2 SW_Push, U1 RP2040, U2 AP2112K-3.3, U3 DRV8833CPWPR, U4 W25Q128JVS, U5 BME280, U6 MCP73831-2-OT, X1 ABM8-272-T3

Commit message: Updated PCB design+schematic
Parts:
- removed C22, C23: 0.1uF, Capacitor_SMD:C_0402_1005Metric, symbol Device:C
- removed J1: USB4235-03-C_REVA, ExternalFootprints:GCT_USB4235-03-C_REVA, symbol USB4235-03-C:USB4235-03-C_REVA
- removed J3: Motor 2, TerminalBlock_Phoenix:TerminalBlock_Phoenix_MKDS-1,5-2-5.08_1x02_P5.08mm_Horizontal, symbol Connector:Screw_Terminal_01x02
- removed J7: Conn_01x15, Connector_PinHeader_2.54mm:PinHeader_1x15_P2.54mm_Vertical, symbol Connector_Generic:Conn_01x15
- removed R16: 4.7k, Resistor_SMD:R_0402_1005Metric, symbol Device:R
- removed U3: DRV8833CPWPR, ExternalFootprints:SOP65P640X120-17N, symbol DRV8833CPWPR:DRV8833CPWPR
- removed U4: W25Q128JVS, Package_SO:SOIC-8_5.3x5.3mm_P1.27mm, symbol Memory_Flash:W25Q128JVS
- removed U5: BME280, Package_LGA:Bosch_LGA-8_2.5x2.5mm_P0.65mm_ClockwisePinNumbering, symbol Sensor:BME280
- added D3, D4: Green, LED_SMD:LED_0603_1608Metric, symbol Device:LED
- added J1: TYPE-C-31-M-12, ExternalFootprints:HRO_TYPE-C-31-M-12, symbol USB_C:TYPE-C-31-M-12
- added J10: BME280 Terminals, TerminalBlock_Phoenix:TerminalBlock_Phoenix_MKDS-1,5-4_1x04_P5.00mm_Horizontal, symbol Connector:Screw_Terminal_01x04
- added J3: Motor 2, Connector_PinHeader_2.54mm:PinHeader_1x02_P2.54mm_Vertical, symbol Connector_Generic:Conn_01x02
- added R14: 330, Resistor_SMD:R_0402_1005Metric, symbol Device:R
- added U3: DRV8833PWP, Package_SO:HTSSOP-16-1EP_4.4x5mm_P0.65mm_EP3.4x5mm_Mask2.46x2.31mm_ThermalVias, symbol Driver_Motor:DRV8833PWP
- added U4: W25Q16JVSS, Package_SON:Winbond_USON-8-1EP_3x2mm_P0.5mm_EP0.2x1.6mm, symbol Memory_Flash:W25Q16JVSS
- C11, C8: value 1uF -> 0.1uF
- C4, C9: value 0.1uF -> 1uF
- D2: footprint LED_SMD:LED_0402_1005Metric -> LED_SMD:LED_0603_1608Metric
- J8: footprint Connector_PinHeader_2.54mm:PinHeader_1x15_P2.54mm_Vertical -> Connector_PinHeader_2.54mm:PinHeader_1x11_P2.54mm_Vertical; symbol Connector_Generic:Conn_01x15 -> Connector_Generic:Conn_01x11
- R11: value 10k -> 470
- R15: value 4.7k -> 500
- R3, R4: value 1 -> 0.2
- U1: footprint Package_DFN_QFN:QFN-56-1EP_7x7mm_P0.4mm_EP3.2x3.2mm -> Package_DFN_QFN:QFN-56-1EP_7x7mm_P0.4mm_EP3.2x3.2mm_ThermalVias
Connections:
- net +1V1: no longer C0.2, C1.2, C10.2, C11.2, C12.2, C13.2, C14.2, C15.2, C16.2, C17.2, C18.2, C19.1, C19.2, C2.2, C20.2, C21.2, C3.2, C4.2, C5.2, C6.2, C7.2, C8.2, C9.2, J4.1, J5.1 (Pin_1), J5.2 (Pin_2), J6.1, J8.14 (Pin_14), J8.15 (Pin_15), J8.3 (Pin_3), Q1.3 (D), R10.2, R12.2, R3.1, R4.1, R6.2, R7.2, SW1.2, SW2.2, U1.19 (TESTEN), U1.57 (GND), U2.2 (GND), U6.2 (V_{SS}), U6.3 (V_{BAT}), X1.2, X1.4
- net +3V3: now also J4.3, J6.3, J8.10 (Pin_10), J8.9 (Pin_9), D3.2 (A), J10.1 (Pin_1), U4.8 (VCC); no longer J4.2, J6.2, J8.1 (Pin_1), R15.1
- net +5V: now also J1.A4_B9 (VBUS), J1.B4_A9 (VBUS); no longer C15.1
- net AIN1: now also U3.16 (AIN1)
- net AIN2: now also U3.15 (AIN2)
- net BIN1: now also U3.9 (BIN1)
- net BIN2: now also U3.10 (BIN2)
- net BME280_SCL: now also U1.31 (GPIO20), J10.4 (Pin_4)
- net BME280_SDA: now also U1.32 (GPIO21), J10.3 (Pin_3); no longer R15.2
- net GPIO15: now also J8.4 (Pin_4)
- net GPIO16: now also J8.5 (Pin_5); no longer J8.4 (Pin_4)
- net GPIO17: now also J8.6 (Pin_6); no longer J8.5 (Pin_5)
- net GPIO18: now also J8.7 (Pin_7); no longer J8.6 (Pin_6)
- net GPIO19: now also J8.8 (Pin_8); no longer J8.7 (Pin_7)
- net GPIO27/ADC1: now also J8.2 (Pin_2); no longer J8.11 (Pin_11)
- net OLED_SCL: now also J6.1; no longer J6.4
- net OLED_SDA: now also J6.2; no longer J6.3
- net QSPI_SCLK: now also U4.6 (CLK)
- net QSPI_SD0: now also U4.5 (DI/IO_{0})
- net QSPI_SD1: now also U4.2 (DO/IO_{1})
- net QSPI_SD2: now also U4.3 (~{WP}/IO_{2})
- net QSPI_SD3: now also U4.7 (~{HOLD}/~{RESET}/IO_{3})
- net QSPI_SS: now also U4.1 (~{CS})
- net USB_D+: now also J1.A6 (DP1), J1.B6 (DP2)
- net USB_D-: now also J1.A7 (DN1), J1.B7 (DN2)
- net nFAULT: now also U3.8 (~{FAULT})
- net nSLEEP: now also U3.1 (~{SLEEP})
- net +MOTORVOLTAGE: now reaches C12.1, D1.1 (K), Q1.2 (S), U2.1 (VIN), U2.3 (EN)
- net +MOTORVOLTAGE: now also C15.1, D4.2 (A), U3.12 (VM)
- net at C14.1: now also U3.14 (VINT)
- net at J2.1 (Pin_1): now also U3.2 (AOUT1)
- net at R3.2: now also U3.3 (AISEN)
- net at J2.2 (Pin_2): now also U3.4 (AOUT2)
- net at R4.2: now also U3.6 (BISEN)
- net at R11.1: now also D2.1 (K); no longer U6.1 (STAT)
- net at R11.2: now also U6.1 (STAT); no longer D2.1 (K)
- net at R7.1: now also J1.B5 (CC2)
- net at R6.1: now also J1.A5 (CC1)
- removed net GPIO20: J8.8 (Pin_8), U1.31 (GPIO20)
- removed net GPIO21: J8.9 (Pin_9), U1.32 (GPIO21)
- net GPIO26/ADC0 renamed GPIO28/ADC0
- net GPIO28/ADC0: now also J8.1 (Pin_1); no longer J8.10 (Pin_10)
- net GPIO28/ADC2 renamed GPIO27/ADC2
- net GPIO27/ADC2: now also J8.3 (Pin_3); no longer J8.12 (Pin_12)
- net GPIO29/ADC3 renamed SOIL_SIG
- net SOIL_SIG: now also J4.1; no longer J8.13 (Pin_13)
- net SOIL_DISABLE renamed GPIO22
- net GPIO22: no longer J4.3
- net SOIL_OUT renamed GND
- net GND: now also C0.2, C1.2, C10.2, C11.2, C12.2, C13.2, C14.2, C15.2, C16.2, C17.2, C18.2, C19.2, C2.2, C20.2, C21.2, C3.2, C4.2, C5.2, C6.2, C7.2, C8.2, C9.2, J5.2 (Pin_2), J6.4, J8.11 (Pin_11), R10.2, R12.2, R15.2, R3.1, R4.1, R6.2, R7.2, SW1.2, SW2.2, U1.19 (TESTEN), U1.57 (GND), U2.2 (GND), U6.2 (V_{SS}), X1.2, X1.4, J1.A1_B12 (GND), J1.B1_A12 (GND), J1.S1 (SHIELD), J1.S2 (SHIELD), J1.S3 (SHIELD), J1.S4 (SHIELD), J10.2 (Pin_2), R14.2, U3.11 (VCP), U3.13 (GND), U3.17 (GND), U4.4 (GND); no longer U1.35 (GPIO23)
- net SWCLK: no longer names the net of U1.24 (SWCLK)
- net SWCLK: no longer J8.2 (Pin_2)
- net SWDIO: no longer names the net of U1.25 (SWDIO)
- new net: D3.1 (K), R14.1
- new net: J3.1 (Pin_1), U3.7 (BOUT1)
- new net: J3.2 (Pin_2), U3.5 (BOUT2)
- new net: D4.1 (K), R15.1
- new net +BATT: C19.1, J5.1 (Pin_1), Q1.3 (D), U6.3 (V_{BAT})
- new net GPIO23: U1.35 (GPIO23)
- no-connect marks 0 -> 5
Other:
- note added: "BME280 Connector"
- note added: "Battery"
- note added: "SIG"
- note added: "Status LEDs"
- note added: "USB-C"
- note added: "Voltage Regulator"
- note removed: "BME280"
- note removed: "DIS"
- note removed: "OUT"
- note removed: "USB/Power"
- moved on the sheet: C0, C1, C12, C13, C15, C16, C17, C18, C19, C2, C21, C3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

Commit message: Finished main PCB
Parts:
- removed C21: 0.1uF, Capacitor_SMD:C_0402_1005Metric, symbol Device:C
- removed SW1: SW_Push, Button_Switch_SMD:SW_Tactile_SPST_NO_Straight_CK_PTS636Sx25SMTRLFS, symbol Switch:SW_Push
- added J7: Conn_01x14, Connector_PinHeader_2.54mm:PinHeader_1x14_P2.54mm_Vertical, symbol Connector_Generic:Conn_01x14
- J6: renamed from J8; value Conn_01x15 -> Conn_01x14; footprint Connector_PinHeader_2.54mm:PinHeader_1x11_P2.54mm_Vertical -> Connector_PinHeader_2.54mm:PinHeader_1x14_P2.54mm_Vertical; symbol Connector_Generic:Conn_01x11 -> Connector_Generic:Conn_01x14
- renumbered J6 to J5, J5 to J8, J10 to J9, SW2 to SW1, U6 to U5
Connections:
- net GPIO22 is gone; now on net nFAULT: U1.34 (GPIO22)
- net GPIO23 is gone; now on net nSLEEP: U1.35 (GPIO23)
- net +3V3: now also J6.11 (Pin_11), J6.12 (Pin_12); no longer J6.9 (Pin_9)
- net GND: now also J6.13 (Pin_13), J6.14 (Pin_14), J7.13 (Pin_13), J7.14 (Pin_14); no longer J6.11 (Pin_11)
- net GPIO0: now also J7.1 (Pin_1)
- net GPIO1: now also J7.2 (Pin_2)
- net GPIO14: now also J7.11 (Pin_11)
- net GPIO15: now also J7.12 (Pin_12); no longer J6.4 (Pin_4)
- net GPIO16: now also J6.7 (Pin_7); no longer J6.5 (Pin_5)
- net GPIO18: now also J6.5 (Pin_5); no longer J6.7 (Pin_7)
- net GPIO19: now also J6.4 (Pin_4); no longer J6.8 (Pin_8)
- net GPIO2: now also J7.3 (Pin_3)
- net GPIO3: now also J7.4 (Pin_4)
- net GPIO6: now also J7.7 (Pin_7)
- net GPIO7: now also J7.8 (Pin_8)
- net GPIO8: now also J7.9 (Pin_9)
- net GPIO9: now also J7.10 (Pin_10)
- net OLED_SCL: now also U1.37 (GPIO25); no longer U1.7 (GPIO5)
- net OLED_SDA: now also U1.36 (GPIO24); no longer U1.6 (GPIO4)
- net nFAULT: no longer U1.37 (GPIO25)
- net nSLEEP: no longer U1.36 (GPIO24)
- net SWCLK: now reaches U1.24 (SWCLK)
- net SWCLK: now also J6.9 (Pin_9)
- net SWDIO: now reaches U1.25 (SWDIO)
- net SWDIO: now also J6.8 (Pin_8)
- net GPIO27/ADC2 renamed GPIO26/ADC0
- net GPIO26/ADC0: now also U1.38 (GPIO26/ADC0); no longer U1.40 (GPIO28/ADC2)
- net GPIO28/ADC0 renamed GPIO28/ADC2
- net GPIO28/ADC2: now also U1.40 (GPIO28/ADC2); no longer U1.38 (GPIO26/ADC0)
- net RUN: no longer names the net of R13.2, U1.26 (RUN)
- new net GPIO4: J7.5 (Pin_5), U1.6 (GPIO4)
- new net GPIO5: J7.6 (Pin_6), U1.7 (GPIO5)
- no-connect marks 5 -> 3
Other:
- note removed: "Reset Button"

Commit message: Finished main PCB
Parts:
- added SW2: SW_Push, Button_Switch_SMD:SW_Tactile_SPST_NO_Straight_CK_PTS636Sx25SMTRLFS, symbol Switch:SW_Push
Connections:
- net GND: now also SW2.2
- net RUN: now reaches R13.2, U1.26 (RUN)
- net RUN: now also SW2.1
Other:
- note added: "Reset Button"
Changed lines of the file:
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@@
 		)
 	)
+	(text "Reset Button\n"
+		(exclude_from_sim no)
+		(at 41.402 26.416 0)
+		(effects
+			(font
+				(size 3.81 3.81)
+				(thickness 0.254)
+				(bold yes)
+			)
+		)
+	)
 	(text "DRV8833 Motor Driver"
 		(exclude_from_sim no)
@@
 	(wire
 		(pts
+			(xy 30.48 48.26) (xy 36.83 48.26)
+		)
+		(stroke
+			(width 0)
+			(type default)
+		)
+	)
+	(wire
+		(pts
+			(xy 46.99 48.26) (xy 49.53 48.26)
+		)
+		(stroke
+			(width 0)
+			(type default)
+		)
+	)
+	(wire
+		(pts
 			(xy 353.06 62.23) (xy 340.36 62.23)
 		)
@@
 	(wire
 		(pts
+			(xy 49.53 48.26) (xy 49.53 50.8)
+		)
+		(stroke
+			(width 0)
+			(type default)
+		)
+	)
+	(wire
+		(pts
 			(xy 189.23 135.89) (xy 203.2 135.89)
 		)
@@
 		)
 	)
+	(label "RUN"
+		(at 118.11 118.11 0)
+		(effects
+			(font
+				(size 1.27 1.27)
+			)
+			(justify left bottom)
+		)
+	)
 	(label "BME280_SDA"
 		(at 203.2 156.21 180)
@@
 		)
 	)
+	(label "RUN"
+		(at 30.48 48.26 0)
+		(effects
+			(font
+				(size 1.27 1.27)
+			)
+			(justify left bottom)
+		)
+	)
 	(label "GPIO16"
 		(at 203.2 143.51 180)
@@
 	(symbol
 		(lib_id "power:GND")
+		(at 49.53 50.8 0)
+		(unit 1)
+		(body_style 1)
+		(exclude_from_sim no)
+		(in_bom yes)
+		(on_board yes)
+		(in_pos_files yes)
+		(dnp no)
+		(fields_autoplaced yes)
+		(property "Reference" "#PWR028"
+			(at 49.53 57.15 0)
+			(hide yes)
+			(show_name no)
+			(do_not_autoplace no)
+			(effects
+				(font
+					(size 1.27 1.27)
+				)
+			)
+		)
+		(property "Value" "GND"
+			(at 49.53 55.88 0)
+			(show_name no)
+			(do_not_autoplace no)
+			(effects
+				(font
+					(size 1.27 1.27)
+				)
+			)
+		)
+		(property "Footprint" ""
+			(at 49.53 50.8 0)
+			(hide yes)
+			(show_name no)
+			(do_not_autoplace no)
+			(effects
+				(font
+					(size 1.27 1.27)
+				)
+			)
+		)
+		(property "Datasheet" ""
+			(at 49.53 50.8 0)
+			(hide yes)
+			(show_name no)
+			(do_not_autoplace no)
+			(effects
+				(font
+					(size 1.27 1.27)
+				)
+			)
+		)
+		(property "Description" "Power symbol creates a global label with name \"GND\" , ground"
+			(at 49.53 50.8 0)
+			(hide yes)
+			(show_name no)
+			(do_not_autoplace no)
+			(effects
+				(font
+					(size 1.27 1.27)
+				)
+			)
+		)
+		(pin "1"
+		)
+		(instances
+			(project "Plant Monitor"
+				(path "/94d2964c-4bbb-42d1-bb87-ec34e272846f"
+					(reference "#PWR028")
+					(unit 1)
+				)
+			)
+		)
+	)
+	(symbol
+		(lib_id "power:GND")
 		(at 364.49 49.53 0)
 		(mirror y)
@@
 					(unit 1)
 				)
+			)
+		)
+	)
+	(symbol
+		(lib_id "Switch:SW_Push")
+		(at 41.91 48.26 0)
+		(unit 1)
+		(body_style 1)
+		(exclude_from_sim no)
+		(in_bom yes)
+		(on_board yes)
+		(in_pos_files yes)
+		(dnp no)
+		(fields_autoplaced yes)
+		(property "Reference" "SW2"
+			(at 41.91 40.64 0)
+			(show_name no)
+			(do_not_autoplace no)
+			(effects
+				(font
+					(size 1.27 1.27)
+				)
+			)
+		)
+		(property "Value" "SW_Push"
+			(at 41.91 43.18 0)
+			(show_name no)
+			(do_not_autoplace no)
+			(effects
+				(font
+					(size 1.27 1.27)
+				)
+			)
+		)
+		(property "Footprint" "Button_Switch_SMD:SW_Tactile_SPST_NO_Straight_CK_PTS636Sx25SMTRLFS"
+			(at 41.91 43.18 0)
+			(hide yes)
+			(show_name no)
+			(do_not_autoplace no)
+			(effects
+				(font
+					(size 1.27 1.27)
+				)
+			)
+		)
+		(property "Datasheet" ""
+			(at 41.91 43.18 0)
+			(hide yes)
+			(show_name no)
+			(do_not_autoplace no)
+			(effects
+				(font
+					(size 1.27 1.27)
+				)
+			)
+		)
+		(property "Description" "Push button switch, generic, two pins"
+			(at 41.91 48.26 0)
+			(hide yes)
+			(show_name no)
+			(do_not_autoplace no)
+			(effects
+				(font
+					(size 1.27 1.27)
+				)
+			)
+		)
+		(pin "1"
+		)
+		(pin "2"
+		)
+		(instances
+			(project "Plant Monitor"
+				(path "/94d2964c-4bbb-42d1-bb87-ec34e272846f"
+					(reference "SW2")
+					(unit 1)
+				)

Commit message: Finished all PCBs, initial CAD complete
Connections:
- net +3V3: now also J9.3 (Pin_3); no longer J9.1 (Pin_1)
- net BME280_SCL: now also J9.2 (Pin_2), U1.32 (GPIO21); no longer J9.4 (Pin_4), U1.31 (GPIO20)
- net BME280_SDA: now also J9.1 (Pin_1), U1.31 (GPIO20); no longer J9.3 (Pin_3), U1.32 (GPIO21)
- net GND: now also J9.4 (Pin_4); no longer J9.2 (Pin_2)
- net at U3.2 (AOUT1): now also J2.2 (Pin_2); no longer J2.1 (Pin_1)
- net at U3.4 (AOUT2): now also J2.1 (Pin_1); no longer J2.2 (Pin_2)
Other:
- moved on the sheet: J2
